File: hover-1 2018250.kicad_sch (KiCad schematic)
At the start: 42 parts, among them Q10 TIP127, Q12 G1, Q14 G1, Q15 G1, Q6 G1, Q9 TIP127, SW1 SW_SPST, U1 GD32F130C8, U5 SOT-223, U6 LM78M05_TO252

Commit message: Add schematic for interupt sensor
Parts:
- added D10: ~, Diode_SMD:D_2010_5025Metric, symbol Device:D
- added R70: 152, Resistor_SMD:R_0603_1608Metric_Pad0.98x0.95mm_HandSolder, symbol Device:R
- added R71: 513, Resistor_SMD:R_0603_1608Metric_Pad0.98x0.95mm_HandSolder, symbol Device:R
- added S1: Everlight_ITR9608-F, OptoDevice:Everlight_ITR9608-F, symbol Sensor_Proximity:ITR9608-F
Connections:
- net 15V: now also D10.2 (A)
- net 3.3V: now also R70.2, R71.1
- net GND: now also S1.2
- net PB12: now reaches U1.25 (PB12)
- new net: R71.2, S1.1
- new net: R70.1, S1.3
Other:
- note added: "Phase driver"
